File: MSPM0-PCB/MSPM0-Project/MSOM0-Project.kicad_pcb (KiCad board)
At the start: 2 copper layers, 58 x 28 mm, 37 parts, among them J1 USB_C_Receptacle_USB2.0_16P, J2 Conn_ARM_SWD_TagConnect_TC2030, U1 MSPM0G3507SPTR, U3 SPX3819M5-L-3-3, U4 CH340E, U5 LIS2DH, X1 8MHz

Commit message: started on the traffic light shield
Other:
- board text added: "MSPM0 learning project"
- board text added: "REV A v. 1.0"
Changed lines of the file:
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@@
 		(layer "Edge.Cuts")
 	)
+	(gr_text "MSPM0 learning project"
+		(at 106.1 89.9 0)
+		(layer "F.SilkS")
+		(effects
+			(font
+				(size 1.5 1)
+				(thickness 0.25)
+			)
+			(justify left bottom)
+		)
+	)
+	(gr_text "REV A\nv. 1.0"
+		(at 87.9 111.8 0)
+		(layer "F.SilkS")
+		(effects
+			(font
+				(size 1 1)
+				(thickness 0.25)
+			)
+			(justify left bottom)
+		)
+	)
 	(segment
 		(start 107.2 100.7)
@@
 			(thermal_gap 0.25)
 			(thermal_bridge_width 0.3)
-			(smoothing fillet)
 		)
 		(polygon
