File: STMTrafficLight/TrafficLight_schem/TrafficLight_connectorpart.kicad_pcb (KiCad board)
At the start: 2 copper layers, 73 parts, among them P1 Conn_01x25, P2 Conn_01x25, P3 Conn_01x25, P4 Conn_01x25, SW1 SW_Push, SW2 SW_Push, SW3 SW_Push, SW4 SW_Push, U1 74HC595D, U2 74HC595D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

Commit message: Added silk screen and edge cutouts
Parts:
- moved P2 261.7 mm to (97.0, 47.8)
- moved P1 260.7 mm to (93.3, 47.8)
- moved P4 228.3 mm to (139.6, 47.8)
- moved P3 227.3 mm to (135.9, 47.8)
Other:
- board outline added: 70 x 140 mm

Commit message: Added silk screen and edge cutouts
Parts:
- removed S1: SW_slide_car, Trafficlight_Library:Sw_slide_car
- added S5: Car 1, Trafficlight_Library:Sw_slide_car, F.Cu at (123.5, 164.4)
- S2: value SW_slide_car -> Car 2
- S3: value SW_slide_car -> Car 3
- S4: value SW_slide_car -> Car 4
- moved SW2 336.8 mm to (96.5, 166.6)
- moved SW1 329.7 mm to (95.9, 127.6)
- moved S2 325.7 mm to (83.4, 152.5), turned to 90 degrees
- moved U2 325.2 mm to (93.0, 138.6), turned to -90 degrees
- moved SW4 325.0 mm to (98.1, 122.1), turned to -90 degrees
- moved U1 307.9 mm to (112.0, 164.3)
- moved LED2 301.9 mm to (96.2, 162.5), turned to 180 degrees
- moved S4 301.1 mm to (114.4, 116.0), turned to 180 degrees
- moved LED6 300.6 mm to (102.6, 155.2)
- moved LED4 299.4 mm to (96.2, 159.7)
- moved LED5 296.7 mm to (102.5, 138.0)
- moved U3 295.6 mm to (135.7, 154.6), turned to 90 degrees
- moved LED1 295.1 mm to (95.8, 131.1), turned to 180 degrees
- moved LED3 294.2 mm to (95.9, 133.6)
- moved LED12 294.0 mm to (105.8, 122.1), turned to 90 degrees
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- renumbered R6 to R12, R9 to R19, R12 to R20, R20 to R3, R19 to R6, R3 to R9
Connections:
- net 595_DS renamed 595_DS_SPI1_MOSI
- net 595_SHCP renamed 595_SHCP_SPI1_CLK
- net 595_STCP renamed 595_STCP_RCLK

Commit message: Added silk screen and edge cutouts
Parts:
- HW status: renamed from LED19
- SW status: renamed from LED23; value Red -> SW status
- moved LED22 322.2 mm to (88.7, 160.6), turned to -90 degrees
- moved LED21 320.2 mm to (91.7, 160.6), turned to -90 degrees
- moved LED7 288.3 mm to (104.4, 114.2), turned to 180 degrees
- moved LED8 287.3 mm to (104.4, 111.1), turned to 180 degrees
- moved LED9 286.5 mm to (104.4, 108.1), turned to 180 degrees
- moved LED24 269.8 mm to (134.2, 161.4)
- moved LED25 269.7 mm to (134.3, 164.2)
- moved LED26 269.7 mm to (134.3, 167.1)
- moved LED16 265.0 mm to (135.0, 132.1), turned to 90 degrees
- moved LED17 261.8 mm to (137.7, 132.1), turned to 90 degrees
- moved LED18 258.5 mm to (140.4, 132.2), turned to 90 degrees
- moved C1 246.5 mm to (131.7, 112.0)
- moved C2 245.4 mm to (131.8, 109.6)
- moved LED20 82.8 mm to (94.7, 160.5), turned to -90 degrees
- moved HW status 38.8 mm to (149.0, 173.3)
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- renumbered D1 to LED24, D2 to LED25, D3 to LED26

Commit message: Added routes and new compontents to solar power
Parts:
- LED19: renamed from HW status
- LED23: renamed from SW status; value SW status -> Red
- S2: value Car 2 -> SW_slide_car
- S3: value Car 3 -> SW_slide_car
- S4: value Car 4 -> SW_slide_car
- S5: value Car 1 -> SW_slide_car
- moved R25 341.2 mm to (85.9, 169.2)
- moved R24 340.8 mm to (86.0, 165.0)
- moved R20 331.4 mm to (85.9, 167.1)
- moved R3 327.1 mm to (86.5, 128.1), turned to 90 degrees
- moved R8 322.1 mm to (102.1, 176.7), turned to 180 degrees
- moved R6 322.0 mm to (102.1, 174.4), turned to 180 degrees
- moved R1 320.0 mm to (86.5, 124.3), turned to 90 degrees
- moved R7 318.4 mm to (86.5, 131.9), turned to 90 degrees
- moved R4 318.0 mm to (86.7, 121.0)
- moved R9 317.7 mm to (86.7, 115.7), turned to 180 degrees
- moved R5 317.3 mm to (86.7, 118.2), turned to 180 degrees
- moved R2 315.6 mm to (102.1, 172.3), turned to 180 degrees
- moved C4 296.3 mm to (93.4, 141.1), turned to 90 degrees
- moved C5 277.2 mm to (117.7, 162.7), turned to 90 degrees
- moved C3 249.3 mm to (146.1, 155.6)
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- renumbered LED24 to D1, LED25 to D2, LED26 to D3
